File: pcb/exposer.kicad_sch (KiCad schematic)
At the start: 10 parts, among them IC1 ULN2065B, J1 Conn_01x04_Female, J2 Conn_01x02, SW1 SW_Push, SW2 SW_Push, SW3 SW_Push, SW4 SW_SPST

Commit message: encoder pcb
Parts:
- removed IC1: ULN2065B, Package_DIP:DIP-16_W7.62mm_LongPads, symbol ULN2065B:ULN2065B
- removed SW1, SW2, SW3: SW_Push, Button_Switch_THT:SW_PUSH_6mm_H5mm, symbol Switch:SW_Push
- added SW1: RotaryEncoder_Switch, Rotary_Encoder:RotaryEncoder_Alps_EC11E-Switch_Vertical_H20mm, symbol Device:RotaryEncoder_Switch
- added U2: ULN2003A, Package_DIP:DIP-16_W7.62mm_LongPads, symbol Transistor_Array:ULN2003A
- BT1: footprint Battery:BatteryHolder_Keystone_1042_1x18650 -> Battery:BatteryHolder_MPD_BH-18650-PC
- J2: footprint Connector_Wire:SolderWirePad_1x02_P7.62mm_Drill2mm -> Connector_Wire:SolderWire-0.75sqmm_1x02_P4.8mm_D1.25mm_OD2.3mm
- SW4: footprint Connector_Molex:Molex_Micro-Fit_3.0_43650-0315_1x03_P3.00mm_Vertical -> Button_Switch_THT:SW_Slide_SPDT_Straight_CK_OS102011MS2Q
Connections:
- net +12V: now also J2.2 (Pin_2); no longer J2.1 (Pin_1)
- net GND: now also SW1.C, SW1.S1, U2.8 (GND)
- net at A1.7 (D4): now also SW1.B
- net at A1.10 (D7): now also U2.1 (I1), U2.2 (I2), U2.3 (I3), U2.4 (I4), U2.5 (I5), U2.6 (I6), U2.7 (I7)
- net at A1.8 (D5): now also SW1.A
- net at A1.9 (D6): now also SW1.S2
- new net: J2.1 (Pin_1), U2.10 (O7), U2.11 (O6), U2.12 (O5), U2.13 (O4), U2.14 (O3), U2.15 (O2), U2.16 (O1)
Other:
- moved on the sheet: J2
