File: rocker_pcb/agitator_pcb/agitator_pcb.kicad_pcb (KiCad board)
At the start: 2 copper layers, 81 x 54.5 mm, 7 parts, among them J1 Conn_01x03_Pin, SW1 SW_DPST_x2

Commit message: model seems fine
Parts:
- moved SW1 2.75 mm to (87.1, 67.0)
Connections:
- A1 pad 19: Net-(A1-A0) -> unconnected-(A1-A0-Pad19)
- A1 pad 20: Net-(A1-A1) -> unconnected-(A1-A1-Pad20)
- A1 pad 23: unconnected-(A1-A4-Pad23) -> Net-(A1-A4)
- A1 pad 24: unconnected-(A1-A5-Pad24) -> Net-(A1-A5)
- RV1 pad 2: Net-(A1-A1) -> Net-(A1-A5)
- RV2 pad 2: Net-(A1-A0) -> Net-(A1-A4)
Routing:
- net +5V: track 202.9 -> 113.2 mm
- net GND: track 169.9 -> 115.8 mm
- net Net-(A1-A1): track 27.3 -> 0.00 mm
- net Net-(A1-A4): track 0.00 -> 19.3 mm
- net Net-(A1-A5): track 0.00 -> 17.8 mm
- net Net-(A1-A0): track 9.87 -> 0.00 mm
- net Net-(A1-D9): track 67.2 -> 59.2 mm
- net +BATT: track 28.4 -> 25.7 mm
- net Net-(BT1-+): track 101.3 -> 98.6 mm
Other:
- board size 81 x 54.5 mm -> 81 x 52.5 mm

Commit message: pcb optimisation
Parts:
- SW1: footprint Button_Switch_SMD:SW_SPDT_CK_JS102011SAQN -> Connector_PinSocket_2.54mm:PinSocket_1x02_P2.54mm_Vertical; moved to F.Cu
- moved SW1 22.3 mm to (91.0, 45.0)
- moved J1 6.00 mm to (76.5, 54.0)
Routing:
- net +BATT: track 25.7 -> 6.04 mm
- net Net-(BT1-+): track 98.6 -> 82.2 mm
- net GND: track 115.8 -> 99.7 mm
- net +5V: track 113.2 -> 106.9 mm
- net Net-(A1-D9): track 59.2 -> 53.2 mm
