File: rocker_pcb/agitator_pcb/agitator_pcb.kicad_sch (KiCad schematic)
At the start: 7 parts, among them J1 Conn_01x03_Pin, SW1 SW_DPST_x2

Commit message: model seems fine
Connections:
- net at RV2.2: now also A1.23 (A4); no longer A1.19 (A0)
- net at RV1.2: now also A1.24 (A5); no longer A1.20 (A1)
Other:
- moved on the sheet: RV1
Changed lines of the file:
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@@
+	(wire
+		(pts
+			(xy 123.19 71.12) (xy 144.78 71.12)
+		)
+		(stroke
+			(width 0)
+			(type default)
+		)
+	)
 	(wire
 		(pts
@@
 	(wire
 		(pts
-			(xy 123.19 58.42) (xy 134.62 58.42)
-		)
-		(stroke
-			(width 0)
-			(type default)
-		)
-	)
-	(wire
-		(pts
 			(xy 90.17 107.95) (xy 121.92 107.95)
 		)
@@
 	(wire
 		(pts
-			(xy 139.7 60.96) (xy 139.7 69.85)
-		)
-		(stroke
-			(width 0)
-			(type default)
-		)
-	)
-	(wire
-		(pts
 			(xy 110.49 83.82) (xy 110.49 90.17)
 		)
@@
 	(wire
 		(pts
-			(xy 134.62 58.42) (xy 134.62 45.72)
+			(xy 123.19 68.58) (xy 134.62 68.58)
+		)
+		(stroke
+			(width 0)
+			(type default)
+		)
+	)
+	(wire
+		(pts
+			(xy 134.62 45.72) (xy 134.62 68.58)
 		)
 		(stroke
@@
 		(pts
 			(xy 115.57 114.3) (xy 115.57 113.03)
-		)
-		(stroke
-			(width 0)
-			(type default)
-		)
-	)
-	(wire
-		(pts
-			(xy 123.19 60.96) (xy 139.7 60.96)
-		)
-		(stroke
-			(width 0)
-			(type default)
-		)
-	)
-	(wire
-		(pts
-			(xy 139.7 69.85) (xy 149.86 69.85)
 		)
 		(stroke
@@
 		(lib_name "GND_5")
 		(lib_id "power:GND")
-		(at 153.67 66.04 180)
+		(at 148.59 67.31 180)
 		(unit 1)
 		(exclude_from_sim no)
@@
 		(fields_autoplaced yes)
 		(property "Reference" "#PWR05"
-			(at 153.67 59.69 0)
+			(at 148.59 60.96 0)
 			(effects
 				(font
@@
 		)
 		(property "Value" "GND"
-			(at 153.67 60.96 0)
+			(at 148.59 62.23 0)
 			(effects
 				(font
@@
 		)
 		(property "Footprint" ""
-			(at 153.67 66.04 0)
+			(at 148.59 67.31 0)
 			(effects
 				(font
@@
 		)
 		(property "Datasheet" ""
-			(at 153.67 66.04 0)
+			(at 148.59 67.31 0)
 			(effects
 				(font
@@
 		)
 		(property "Description" ""
-			(at 153.67 66.04 0)
+			(at 148.59 67.31 0)
 			(effects
 				(font
@@
 	(symbol
 		(lib_id "Device:R_Potentiometer")
-		(at 153.67 69.85 180)
+		(at 148.59 71.12 180)
 		(unit 1)
 		(exclude_from_sim no)
@@
 		(fields_autoplaced yes)
 		(property "Reference" "RV1"
-			(at 156.21 71.1201 0)
+			(at 151.13 72.3901 0)
 			(effects
 				(font
@@
 		)
 		(property "Value" "R_Potentiometer"
-			(at 156.21 68.5801 0)
+			(at 151.13 69.8501 0)
 			(effects
 				(font
@@
 		)
 		(property "Footprint" "Potentiometer_THT:Potentiometer_Piher_T-16H_Single_Horizontal"
-			(at 153.67 69.85 0)
+			(at 148.59 71.12 0)
 			(effects
 				(font
@@
 		)
 		(property "Datasheet" "~"
-			(at 153.67 69.85 0)
+			(at 148.59 71.12 0)
 			(effects
 				(font
@@
 		)
 		(property "Description" "Potentiometer"
-			(at 153.67 69.85 0)
+			(at 148.59 71.12 0)
 			(effects
 				(font
@@
 		(lib_name "+12V_4")
 		(lib_id "power:+12V")
-		(at 153.67 73.66 180)
+		(at 148.59 74.93 180)
 		(unit 1)
 		(exclude_from_sim no)
@@
 		(fields_autoplaced yes)
 		(property "Reference" "#PWR04"
-			(at 153.67 69.85 0)
+			(at 148.59 71.12 0)
 			(effects
 				(font
@@
 		)
 		(property "Value" "+5V"
-			(at 153.67 77.47 0)
+			(at 148.59 78.74 0)
 			(effects
 				(font
@@
 		)
 		(property "Footprint" ""
-			(at 153.67 73.66 0)
+			(at 148.59 74.93 0)
 			(effects
 				(font
@@
 		)
 		(property "Datasheet" ""
-			(at 153.67 73.66 0)
+			(at 148.59 74.93 0)
 			(effects
 				(font
@@
 		)
 		(property "Description" ""
-			(at 153.67 73.66 0)
-			(effects
-				(font
+			(at 148.59 74.93 0)
+			(effects
+				(font

Commit message: pcb optimisation
Parts:
- SW1: footprint Button_Switch_SMD:SW_SPDT_CK_JS102011SAQN -> Connector_PinSocket_2.54mm:PinSocket_1x02_P2.54mm_Vertical
Changed lines of the file:
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@@
 			)
 		)
-		(property "Footprint" "Button_Switch_SMD:SW_SPDT_CK_JS102011SAQN"
+		(property "Footprint" "Connector_PinSocket_2.54mm:PinSocket_1x02_P2.54mm_Vertical"
 			(at 54.61 69.85 0)
 			(effects
